File: circuits/LED Dice v3/LED Dice/LED Dice.kicad_sch (KiCad schematic)
At the start: 0 parts

Commit message: schematic is complete
Other:
- sheet Microcontroller ports: added +3.3V, DinLED, GND, USBD+, USBD-, Vsample; removed none
- sheet Power and Comms ports: added +3.3V, +5V, GND, USB D+, USB D-, Vsense; removed none
