File: circuits/LED Dice v3/LED Dice/led matrix.kicad_sch (KiCad schematic)
At the start: 7 parts

Commit message: layout progress
Parts:
- D1, D2, D3, D4, D5, D6, D7: footprint LED_SMD:LED_WS2812B_PLCC4_5.0x5.0mm_P3.2mm -> LEDs:LED_WS2812B_PLCC4_5.0x5.0mm_P3.2mm
Changed lines of the file:
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@@
 			)
 		)
-		(property "Footprint" "LED_SMD:LED_WS2812B_PLCC4_5.0x5.0mm_P3.2mm"
+		(property "Footprint" "LEDs:LED_WS2812B_PLCC4_5.0x5.0mm_P3.2mm"
 			(at 91.44 64.77 0)
 			(hide yes)
@@
 			)
 		)
-		(property "Footprint" "LED_SMD:LED_WS2812B_PLCC4_5.0x5.0mm_P3.2mm"
+		(property "Footprint" "LEDs:LED_WS2812B_PLCC4_5.0x5.0mm_P3.2mm"
 			(at 163.83 105.41 0)
 			(hide yes)
@@
 			)
 		)
-		(property "Footprint" "LED_SMD:LED_WS2812B_PLCC4_5.0x5.0mm_P3.2mm"
+		(property "Footprint" "LEDs:LED_WS2812B_PLCC4_5.0x5.0mm_P3.2mm"
 			(at 91.44 105.41 0)
 			(hide yes)
@@
 			)
 		)
-		(property "Footprint" "LED_SMD:LED_WS2812B_PLCC4_5.0x5.0mm_P3.2mm"
+		(property "Footprint" "LEDs:LED_WS2812B_PLCC4_5.0x5.0mm_P3.2mm"
 			(at 165.1 143.51 0)
 			(hide yes)
@@
 			)
 		)
-		(property "Footprint" "LED_SMD:LED_WS2812B_PLCC4_5.0x5.0mm_P3.2mm"
+		(property "Footprint" "LEDs:LED_WS2812B_PLCC4_5.0x5.0mm_P3.2mm"
 			(at 128.27 105.41 0)
 			(hide yes)
@@
 			)
 		)
-		(property "Footprint" "LED_SMD:LED_WS2812B_PLCC4_5.0x5.0mm_P3.2mm"
+		(property "Footprint" "LEDs:LED_WS2812B_PLCC4_5.0x5.0mm_P3.2mm"
 			(at 91.44 143.51 0)
 			(hide yes)
@@
 			)
 		)
-		(property "Footprint" "LED_SMD:LED_WS2812B_PLCC4_5.0x5.0mm_P3.2mm"
+		(property "Footprint" "LEDs:LED_WS2812B_PLCC4_5.0x5.0mm_P3.2mm"
 			(at 163.83 64.77 0)
 			(hide yes)
